Commit message: fix file path

File: urdf/robot_description.urdf (robot description, URDF)
Before this commit: robot NanoRobot, 8 links, 7 joints
Links:
- link ball_wheel_link: geometry collision mesh filename=package://nanorobot_description/meshes/ball_wheel_link.STL; visual mesh filename=package://nanorobot_description/meshes/ball_wheel_link.STL
- link base_camera_link: geometry collision mesh filename=package://nanorobot_description/meshes/base_camera_link.STL; visual mesh filename=package://nanorobot_description/meshes/base_camera_link.STL
- link base_laser_link: geometry collision mesh filename=package://nanorobot_description/meshes/base_laser_link.STL; visual mesh filename=package://nanorobot_description/meshes/base_laser_link.STL
- link base_link: geometry collision mesh filename=package://nanorobot_description/meshes/base_link.STL; visual mesh filename=package://nanorobot_description/meshes/base_link.STL
- link imu: geometry collision mesh filename=package://nanorobot_description/meshes/imu.STL; visual mesh filename=package://nanorobot_description/meshes/imu.STL
- link left_wheel_link: geometry collision mesh filename=package://nanorobot_description/meshes/left_wheel_link.STL; visual mesh filename=package://nanorobot_description/meshes/left_wheel_link.STL
- link right_wheel_link: geometry collision mesh filename=package://nanorobot_description/meshes/right_wheel_link.STL; visual mesh filename=package://nanorobot_description/meshes/right_wheel_link.STL

File: urdf/robot_description.urdf.xacro (robot description, xacro)
@@ -2,5 +2,5 @@
 <robot name="NanoRobot"  xmlns:xacro="http://ros.org/wiki/xacro">
   <xacro:arg name="robot_name" default=""/>
-  <xacro:include filename="$(find robot_description)/urdf/robot_description.gazebo.xacro" />
+  <xacro:include filename="$(find nanorobot_description)/urdf/robot_description.gazebo.xacro" />
   <link name="$(arg robot_name)/base_footprint"/>
   <joint name="base_joint" type="fixed">
@@ -31,19 +31,19 @@
       <geometry>
         <mesh
-          filename="package://robot_description/meshes/base_link.STL" />
-      </geometry>
-      <material
-        name="">
-        <color
-          rgba="1 1 1 1" />
-      </material>
-    </visual>
-    <collision>
-      <origin
-        xyz="0 0 0"
-        rpy="0 0 0" />
-      <geometry>
-        <mesh
-          filename="package://robot_description/meshes/base_link.STL" />
+          filename="package://nanorobot_description/meshes/base_link.STL" />
+      </geometry>
+      <material
+        name="">
+        <color
+          rgba="1 1 1 1" />
+      </material>
+    </visual>
+    <collision>
+      <origin
+        xyz="0 0 0"
+        rpy="0 0 0" />
+      <geometry>
+        <mesh
+          filename="package://nanorobot_description/meshes/base_link.STL" />
       </geometry>
     </collision>
@@ -71,19 +71,19 @@
       <geometry>
         <mesh
-          filename="package://robot_description/meshes/imu.STL" />
-      </geometry>
-      <material
-        name="">
-        <color
-          rgba="1 1 1 1" />
-      </material>
-    </visual>
-    <collision>
-      <origin
-        xyz="0 0 0"
-        rpy="0 0 0" />
-      <geometry>
-        <mesh
-          filename="package://robot_description/meshes/imu.STL" />
+          filename="package://nanorobot_description/meshes/imu.STL" />
+      </geometry>
+      <material
+        name="">
+        <color
+          rgba="1 1 1 1" />
+      </material>
+    </visual>
+    <collision>
+      <origin
+        xyz="0 0 0"
+        rpy="0 0 0" />
+      <geometry>
+        <mesh
+          filename="package://nanorobot_description/meshes/imu.STL" />
       </geometry>
     </collision>
@@ -124,19 +124,19 @@
       <geometry>
         <mesh
-          filename="package://robot_description/meshes/base_camera_link.STL" />
-      </geometry>
-      <material
-        name="">
-        <color
-          rgba="1 1 1 1" />
-      </material>
-    </visual>
-    <collision>
-      <origin
-        xyz="0 0 0"
-        rpy="0 0 0" />
-      <geometry>
-        <mesh
-          filename="package://robot_description/meshes/base_camera_link.STL" />
+          filename="package://nanorobot_description/meshes/base_camera_link.STL" />
+      </geometry>
+      <material
+        name="">
+        <color
+          rgba="1 1 1 1" />
+      </material>
+    </visual>
+    <collision>
+      <origin
+        xyz="0 0 0"
+        rpy="0 0 0" />
+      <geometry>
+        <mesh
+          filename="package://nanorobot_description/meshes/base_camera_link.STL" />
       </geometry>
     </collision>
@@ -177,19 +177,19 @@
       <geometry>
         <mesh
-          filename="package://robot_description/meshes/base_laser_link.STL" />
-      </geometry>
-      <material
-        name="">
-        <color
-          rgba="1 1 1 1" />
-      </material>
-    </visual>
-    <collision>
-      <origin
-        xyz="0 0 0"
-        rpy="0 0 0" />
-      <geometry>
-        <mesh
-          filename="package://robot_description/meshes/base_laser_link.STL" />
+          filename="package://nanorobot_description/meshes/base_laser_link.STL" />
+      </geometry>
+      <material
+        name="">
+        <color
+          rgba="1 1 1 1" />
+      </material>
+    </visual>
+    <collision>
+      <origin
+        xyz="0 0 0"
+        rpy="0 0 0" />
+      <geometry>
+        <mesh
+          filename="package://nanorobot_description/meshes/base_laser_link.STL" />
       </geometry>
     </collision>
@@ -230,5 +230,5 @@
       <geometry>
         <mesh
-          filename="package://robot_description/meshes/left_wheel_link.STL" />
+          filename="package://nanorobot_description/meshes/left_wheel_link.STL" />
       </geometry>
       <material
@@ -244,5 +244,5 @@
       <geometry>
         <mesh
-          filename="package://robot_description/meshes/left_wheel_link.STL" />
+          filename="package://nanorobot_description/meshes/left_wheel_link.STL" />
       </geometry>
     </collision>
@@ -286,5 +286,5 @@
       <geometry>
         <mesh
-          filename="package://robot_description/meshes/right_wheel_link.STL" />
+          filename="package://nanorobot_description/meshes/right_wheel_link.STL" />
       </geometry>
       <material
@@ -300,5 +300,5 @@
       <geometry>
         <mesh
-          filename="package://robot_description/meshes/right_wheel_link.STL" />
+          filename="package://nanorobot_description/meshes/right_wheel_link.STL" />
       </geometry>
     </collision>
@@ -342,19 +342,19 @@
       <geometry>
         <mesh
-          filename="package://robot_description/meshes/ball_wheel_link.STL" />
-      </geometry>
-      <material
-        name="">
-        <color
-          rgba="1 1 1 1" />
-      </material>
-    </visual>
-    <collision>
-      <origin
-        xyz="0 0 0"
-        rpy="0 0 0" />
-      <geometry>
-        <mesh
-          filename="package://robot_description/meshes/ball_wheel_link.STL" />
+          filename="package://nanorobot_description/meshes/ball_wheel_link.STL" />
+      </geometry>
+      <material
+        name="">
+        <color
+          rgba="1 1 1 1" />
+      </material>
+    </visual>
+    <collision>
+      <origin
+        xyz="0 0 0"
+        rpy="0 0 0" />
+      <geometry>
+        <mesh
+          filename="package://nanorobot_description/meshes/ball_wheel_link.STL" />
       </geometry>
     </collision>
