Commit message: fix mu param

File: urdf/robot_description.gazebo.xacro (robot description, xacro)
@@ -9,6 +9,6 @@
   </gazebo>
   <gazebo reference="$(arg robot_name)/left_wheel_link">
-    <mu1>0.5</mu1>
-    <mu2>0.5</mu2>
+    <mu1>5</mu1>
+    <mu2>5</mu2>
     <kp>500000.0</kp>
     <kd>10.0</kd>
@@ -19,6 +19,6 @@
   </gazebo>
   <gazebo reference="$(arg robot_name)/right_wheel_link">
-    <mu1>0.5</mu1>
-    <mu2>0.5</mu2>
+    <mu1>5</mu1>
+    <mu2>5</mu2>
     <kp>500000.0</kp>
     <kd>10.0</kd>
@@ -56,5 +56,5 @@
       <publishWheelJointState>true</publishWheelJointState>
       <legacyMode>false</legacyMode>
-      <updateRate>30</updateRate>
+      <updateRate>50</updateRate>
       <leftJoint>left_wheel_joint</leftJoint>
       <rightJoint>right_wheel_joint</rightJoint>

File: urdf/robot_description.urdf (robot description, URDF)
Before this commit: robot NanoRobot, 8 links, 7 joints
Links:
- link ball_wheel_link: mass 0.00218512482182764 -> 1.00218512482182764
- link base_laser_link: mass 0.4442754144754 -> 0.0442754144754
- link base_link: mass 0.4442754144754 -> 0.1442754144754

Commit message: Initial commit: robot simulation package

File: urdf/robot_description.gazebo.xacro (robot description, xacro)
@@ -1,12 +1,12 @@
 <?xml version="1.0"?>
 <robot name="NanoRobot" xmlns:xacro="http://ros.org/wiki/xacro">
-  <xacro:arg name="laser_visual" default="false"/>
+  <xacro:arg name="laser_visual" default="true"/>
   <xacro:arg name="camera_visual" default="false"/>
   <xacro:arg name="imu_visual"   default="false"/>
   <xacro:arg name="robot_name" default=""/>
-  <gazebo reference="$(arg robot_name)/base_link">
+  <gazebo reference="base_link">
     <material>Gazebo/DarkGrey</material>
   </gazebo>
-  <gazebo reference="$(arg robot_name)/left_wheel_link">
+  <gazebo reference="left_wheel_link">
     <mu1>5</mu1>
     <mu2>5</mu2>
@@ -18,5 +18,5 @@
     <material>Gazebo/FlatBlack</material>
   </gazebo>
-  <gazebo reference="$(arg robot_name)/right_wheel_link">
+  <gazebo reference="right_wheel_link">
     <mu1>5</mu1>
     <mu2>5</mu2>
@@ -28,5 +28,5 @@
     <material>Gazebo/FlatBlack</material>
   </gazebo>
-  <gazebo reference="$(arg robot_name)/ball_wheel_link">
+  <gazebo reference="ball_wheel_link">
     <mu1>0.1</mu1>
     <mu2>0.1</mu2>
@@ -37,5 +37,5 @@
     <material>Gazebo/FlatBlack</material>
   </gazebo>
-  <gazebo reference="$(arg robot_name)/imu">
+  <gazebo reference="imu">
     <sensor type="imu" name="imu">
       <always_on>true</always_on>
@@ -69,5 +69,5 @@
     <plugin name="imu_plugin" filename="libgazebo_ros_imu.so">
       <alwaysOn>true</alwaysOn>
-      <bodyName>$(arg robot_name)/imu</bodyName>
+      <bodyName>imu</bodyName>
       <frameName>imu</frameName>
       <topicName>imu</topicName>
@@ -94,5 +94,5 @@
     </plugin>
   </gazebo>
-  <gazebo reference="$(arg robot_name)/base_laser_link">
+  <gazebo reference="base_laser_link">
     <material>Gazebo/FlatBlack</material>
     <sensor type="ray" name="rplidar_sensor">
@@ -100,8 +100,10 @@
       <visualize>$(arg laser_visual)</visualize>
       <update_rate>7</update_rate>
+      <!-- <update_rate>10</update_rate> -->
       <ray>
         <scan>
           <horizontal>
             <samples>720</samples>
+            <!-- <resolution>1.0</resolution> -->
             <resolution>0.5</resolution>
             <min_angle>0.0</min_angle>
@@ -111,5 +113,5 @@
         <range>
           <min>0.120</min>
-          <max>12.0</max>
+          <max>8.0</max>
           <resolution>0.015</resolution>
         </range>
@@ -126,6 +128,6 @@
     </sensor>
   </gazebo>
-  <gazebo reference="$(arg robot_name)/base_camera_link">
-    <sensor type="camera" name="csi Camera">
+  <gazebo reference="base_camera_link">
+    <sensor type="camera" name="csi_camera">
       <always_on>true</always_on>
       <visualize>$(arg camera_visual)</visualize>
@@ -145,5 +147,5 @@
         <alwaysOn>true</alwaysOn>
         <updateRate>30.0</updateRate>
-        <cameraName>/</cameraName>
+        <cameraName>camera</cameraName>
         <frameName>base_camera_link</frameName>
         <imageTopicName>image_raw</imageTopicName>

File: urdf/robot_description.urdf.xacro (robot description, xacro)
@@ -3,12 +3,12 @@
   <xacro:arg name="robot_name" default=""/>
   <xacro:include filename="$(find nanorobot_description)/urdf/robot_description.gazebo.xacro" />
-  <link name="$(arg robot_name)/base_footprint"/>
+  <link name="base_footprint"/>
   <joint name="base_joint" type="fixed">
-    <parent link="$(arg robot_name)/base_footprint"/>
-    <child link="$(arg robot_name)/base_link"/>
+    <parent link="base_footprint"/>
+    <child link="base_link"/>
     <origin xyz="0.0 0.0 0.012" rpy="0 0 0"/>
   </joint>
   <link
-    name="$(arg robot_name)/base_link">
+    name="base_link">
     <inertial>
       <origin
@@ -50,5 +50,5 @@
   </link>
   <link
-    name="$(arg robot_name)/imu">
+    name="imu">
     <inertial>
       <origin
@@ -96,12 +96,12 @@
       rpy="0 5.2369E-16 0" />
     <parent
-      link="$(arg robot_name)/base_link" />
-    <child
-      link="$(arg robot_name)/imu" />
+      link="base_link" />
+    <child
+      link="imu" />
     <axis
       xyz="0 0 0" />
   </joint>
   <link
-    name="$(arg robot_name)/base_camera_link">
+    name="base_camera_link">
     <inertial>
       <origin
@@ -149,12 +149,12 @@
       rpy="-2.2337E-16 0.2 0" />
     <parent
-      link="$(arg robot_name)/base_link" />
-    <child
-      link="$(arg robot_name)/base_camera_link" />
+      link="base_link" />
+    <child
+      link="base_camera_link" />
     <axis
       xyz="0 0 0" />
   </joint>
   <link
-    name="$(arg robot_name)/base_laser_link">
+    name="base_laser_link">
     <inertial>
       <origin
@@ -202,12 +202,12 @@
       rpy="-1.6843E-15 -1.0776E-15 4.3793E-15" />
     <parent
-      link="$(arg robot_name)/base_link" />
-    <child
-      link="$(arg robot_name)/base_laser_link" />
+      link="base_link" />
+    <child
+      link="base_laser_link" />
     <axis
       xyz="0 0 0" />
   </joint>
   <link
-    name="$(arg robot_name)/left_wheel_link">
+    name="left_wheel_link">
     <inertial>
       <origin
@@ -255,7 +255,7 @@
       rpy="-1.5708 5.2369E-16 8.6736E-17" />
     <parent
-      link="$(arg robot_name)/base_link" />
-    <child
-      link="$(arg robot_name)/left_wheel_link" />
+      link="base_link" />
+    <child
+      link="left_wheel_link" />
     <axis
       xyz="0 0 1" />
@@ -265,5 +265,5 @@
   </joint>
   <link
-    name="$(arg robot_name)/right_wheel_link">
+    name="right_wheel_link">
     <inertial>
       <origin
@@ -311,7 +311,7 @@
       rpy="1.5708 -5.2369E-16 3.1416" />
     <parent
-      link="$(arg robot_name)/base_link" />
-    <child
-      link="$(arg robot_name)/right_wheel_link" />
+      link="base_link" />
+    <child
+      link="right_wheel_link" />
     <axis
       xyz="0 0 1" />
@@ -321,5 +321,5 @@
   </joint>
   <link
-    name="$(arg robot_name)/ball_wheel_link">
+    name="ball_wheel_link">
     <inertial>
       <origin
@@ -367,7 +367,7 @@
       rpy="0 5.2369E-16 0" />
     <parent
-      link="$(arg robot_name)/base_link" />
-    <child
-      link="$(arg robot_name)/ball_wheel_link" />
+      link="base_link" />
+    <child
+      link="ball_wheel_link" />
     <axis
       xyz="0 0 0" />
